File: viztisztito.kicad_pcb (KiCad board)
At the start: 2 copper layers, 74 parts, among them P1 WATER_LEVEL_CONN, P10 CONN_01X01, P11 CONN_01X01, P12 CONN_01X01, P13 CONN_01X01, P14 CONN_01X02, P2 BOARD_CONN, P4 CONN_01X03, P6 CONN_01X02, P7 CONN_01X02, P8 CONN_01X02, P9 CONN_01X10, Q1 BC850, T1 TRANSFO, U1 SPX2920M3-3.3, U10 ACS722, U2 LTV-847, U3 SHARPS202S02, U4 ACS716, U5 MCP3004, U6 TC77, U7 SPX2920M3-3.3, U8 SPX2920M3-3.3, U9 SPX2920M3-3.3

Commit message: some minor changes
Routing:
- net Net-(D6-Pad1): track 27.9 -> 31.7 mm
- net /SSR_N_SENSING/FAULT_EN: track 53.2 -> 52.2 mm
- net GNDREF: track 152.2 -> 151.2 mm
Changed lines of the file:
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@@
   (segment (start 151.788 153.932) (end 151.788 150.932) (width 0.6096) (layer F.Cu) (net 3))
   (segment (start 151.788 156.932) (end 151.788 153.932) (width 0.6096) (layer F.Cu) (net 3))
+  (segment (start 69.420849 148.041757) (end 77.75 148.041757) (width 0.6096) (layer F.Cu) (net 4))
+  (segment (start 67.879092 146.5) (end 69.420849 148.041757) (width 0.6096) (layer F.Cu) (net 4))
+  (segment (start 60 146.5) (end 67.879092 146.5) (width 0.6096) (layer F.Cu) (net 4))
   (segment (start 125.5 173.04) (end 125.5 176) (width 0.8128) (layer B.Cu) (net 4))
   (via (at 125.5 176) (size 2) (drill 0.8) (layers F.Cu B.Cu) (net 4))
@@
   (segment (start 79.291757 146.5) (end 83 146.5) (width 0.6096) (layer F.Cu) (net 4))
   (segment (start 77.75 148.041757) (end 77.812961 148.041757) (width 0.6096) (layer F.Cu) (net 4))
-  (segment (start 73.914023 148.041757) (end 77.75 148.041757) (width 0.6096) (layer F.Cu) (net 4))
-  (segment (start 72.70578 149.25) (end 73.914023 148.041757) (width 0.6096) (layer F.Cu) (net 4))
-  (segment (start 64.260144 149.25) (end 72.70578 149.25) (width 0.6096) (layer F.Cu) (net 4))
-  (segment (start 62.355535 147.345391) (end 64.260144 149.25) (width 0.6096) (layer F.Cu) (net 4))
-  (segment (start 60 146.5) (end 61.510144 146.5) (width 0.6096) (layer F.Cu) (net 4))
-  (segment (start 61.510144 146.5) (end 62.355535 147.345391) (width 0.6096) (layer F.Cu) (net 4))
   (segment (start 87.928 162.56) (end 86.3184 162.56) (width 0.6096) (layer F.Cu) (net 4))
   (segment (start 86.3184 162.56) (end 85.988199 162.229799) (width 0.6096) (layer F.Cu) (net 4))
@@
   (via (at 149.75 167.43981) (size 2) (drill 0.8) (layers F.Cu B.Cu) (net 21))
   (segment (start 146.524 171.324) (end 146.524 176.524) (width 2.54) (layer B.Cu) (net 21))
-  (segment (start 63.25 139.5) (end 68.885 139.5) (width 0.8128) (layer F.Cu) (net 22))
-  (segment (start 68.885 139.5) (end 69.5 140.115) (width 0.8128) (layer F.Cu) (net 22))
-  (segment (start 60.198 140.97) (end 61.78 140.97) (width 0.8128) (layer B.Cu) (net 22))
-  (segment (start 61.78 140.97) (end 63.25 139.5) (width 0.8128) (layer B.Cu) (net 22))
-  (via (at 63.25 139.5) (size 2) (drill 0.8) (layers F.Cu B.Cu) (net 22))
+  (segment (start 65.280006 140.97) (end 66.25 140.000006) (width 0.8128) (layer B.Cu) (net 22))
+  (segment (start 60.198 140.97) (end 65.280006 140.97) (width 0.8128) (layer B.Cu) (net 22))
+  (segment (start 66.364994 140.115) (end 66.25 140.000006) (width 0.8128) (layer F.Cu) (net 22))
+  (segment (start 69.5 140.115) (end 66.364994 140.115) (width 0.8128) (layer F.Cu) (net 22))
+  (via (at 66.25 140.000006) (size 2) (drill 0.8) (layers F.Cu B.Cu) (net 22))
   (segment (start 71.50102 141) (end 70.385 141) (width 0.8128) (layer F.Cu) (net 22))
   (segment (start 70.385 141) (end 69.5 140.115) (width 0.8128) (layer F.Cu) (net 22))
-  (segment (start 57.5 144.25) (end 58.914213 144.25) (width 0.8128) (layer F.Cu) (net 23))
-  (segment (start 58.914213 144.25) (end 59.652803 143.51141) (width 0.8128) (layer F.Cu) (net 23))
-  (segment (start 59.652803 143.51141) (end 67.95079 143.51141) (width 0.8128) (layer F.Cu) (net 23))
-  (segment (start 67.95079 143.51141) (end 68.0772 143.385) (width 0.8128) (layer F.Cu) (net 23))
-  (segment (start 68.0772 143.385) (end 69.5 143.385) (width 0.8128) (layer F.Cu) (net 23))
-  (segment (start 57.658 140.97) (end 57.658 144.092) (width 0.8128) (layer B.Cu) (net 23))
-  (segment (start 57.658 144.092) (end 57.5 144.25) (width 0.8128) (layer B.Cu) (net 23))
-  (via (at 57.5 144.25) (size 2) (drill 0.8) (layers F.Cu B.Cu) (net 23))
+  (segment (start 57.658 140.97) (end 57.658 142.158) (width 0.8128) (layer B.Cu) (net 23))
+  (segment (start 57.658 142.158) (end 59 143.5) (width 0.8128) (layer B.Cu) (net 23))
+  (segment (start 59 143.5) (end 59.439594 143.5) (width 0.8128) (layer B.Cu) (net 23))
+  (segment (start 70.085793 145.5) (end 71.500006 145.5) (width 0.8128) (layer B.Cu) (net 23))
+  (segment (start 59.439594 143.5) (end 59.451004 143.51141) (width 0.8128) (layer B.Cu) (net 23))
+  (segment (start 59.451004 143.51141) (end 60.944996 143.51141) (width 0.8128) (layer B.Cu) (net 23))
+  (segment (start 60.944996 143.51141) (end 60.956406 143.5) (width 0.8128) (layer B.Cu) (net 23))
+  (segment (start 60.956406 143.5) (end 68.085793 143.5) (width 0.8128) (layer B.Cu) (net 23))
+  (segment (start 68.085793 143.5) (end 70.085793 145.5) (width 0.8128) (layer B.Cu) (net 23))
+  (segment (start 71.500006 145.230006) (end 71.500006 145.5) (width 0.8128) (layer F.Cu) (net 23))
+  (segment (start 69.655 143.385) (end 71.500006 145.230006) (width 0.8128) (layer F.Cu) (net 23))
+  (segment (start 69.5 143.385) (end 69.655 143.385) (width 0.8128) (layer F.Cu) (net 23))
+  (via (at 71.500006 145.5) (size 2) (drill 0.8) (layers F.Cu B.Cu) (net 23))
   (segment (start 69.5 143.385) (end 70.7196 143.385) (width 0.6096) (layer F.Cu) (net 23))
   (segment (start 70.7196 143.385) (end 70.8346 143.5) (width 0.6096) (layer F.Cu) (net 23))
@@
   (segment (start 84.749996 145) (end 84.999996 145.25) (width 0.6096) (layer F.Cu) (net 44))
   (via (at 84.999996 145.25) (size 2) (drill 0.8) (layers F.Cu B.Cu) (net 44))
+  (segment (start 81.848969 147.825245) (end 82.65583 148.632106) (width 0.6096) (layer F.Cu) (net 46))
+  (segment (start 78.328495 149.286367) (end 79.789617 147.825245) (width 0.6096) (layer F.Cu) (net 46))
+  (segment (start 62.27801 149.286368) (end 78.328495 149.286367) (width 0.6096) (layer F.Cu) (net 46))
+  (segment (start 61.676055 148.684413) (end 62.27801 149.286368) (width 0.6096) (layer F.Cu) (net 46))
+  (segment (start 61.30336 148.684413) (end 61.676055 148.684413) (width 0.6096) (layer F.Cu) (net 46))
+  (segment (start 61.179146 148.560199) (end 61.30336 148.684413) (width 0.6096) (layer F.Cu) (net 46))
+  (segment (start 82.65583 148.632106) (end 83.655829 149.632105) (width 0.6096) (layer F.Cu) (net 46))
+  (segment (start 54.458 148.59) (end 56.1926 148.59) (width 0.6096) (layer F.Cu) (net 46))
+  (segment (start 56.222401 148.560199) (end 61.179146 148.560199) (width 0.6096) (layer F.Cu) (net 46))
+  (segment (start 79.789617 147.825245) (end 81.848969 147.825245) (width 0.6096) (layer F.Cu) (net 46))
+  (segment (start 56.1926 148.59) (end 56.222401 148.560199) (width 0.6096) (layer F.Cu) (net 46))
   (segment (start 83.655829 149.632105) (end 83.655829 168.074515) (width 0.6096) (layer B.Cu) (net 46))
   (segment (start 83.655829 168.074515) (end 84.86 169.278686) (width 0.6096) (layer B.Cu) (net 46))
   (segment (start 84.86 169.278686) (end 84.86 170.5) (width 0.6096) (layer B.Cu) (net 46))
-  (segment (start 61.84 148.59) (end 63.75539 150.50539) (width 0.6096) (layer F.Cu) (net 46))
-  (segment (start 63.75539 150.50539) (end 73.210534 150.50539) (width 0.6096) (layer F.Cu) (net 46))
-  (segment (start 54.458 148.59) (end 58.418358 148.59) (width 0.6096) (layer F.Cu) (net 46))
-  (segment (start 58.418358 148.59) (end 58.448159 148.560199) (width 0.6096) (layer F.Cu) (net 46))
-  (segment (start 58.448159 148.560199) (end 61.551841 148.560199) (width 0.6096) (layer F.Cu) (net 46))
-  (segment (start 61.551841 148.560199) (end 61.581642 148.59) (width 0.6096) (layer F.Cu) (net 46))
-  (segment (start 61.581642 148.59) (end 61.84 148.59) (width 0.6096) (layer F.Cu) (net 46))
-  (segment (start 73.210534 150.50539) (end 74.429557 149.286367) (width 0.6096) (layer F.Cu) (net 46))
-  (segment (start 74.429557 149.286367) (end 78.328495 149.286367) (width 0.6096) (layer F.Cu) (net 46))
-  (segment (start 78.328495 149.286367) (end 79.789617 147.825245) (width 0.6096) (layer F.Cu) (net 46))
-  (segment (start 79.789617 147.825245) (end 81.848969 147.825245) (width 0.6096) (layer F.Cu) (net 46))
-  (segment (start 81.848969 147.825245) (end 82.65583 148.632106) (width 0.6096) (layer F.Cu) (net 46))
-  (segment (start 82.65583 148.632106) (end 83.655829 149.632105) (width 0.6096) (layer F.Cu) (net 46))
   (via (at 83.655829 149.632105) (size 2) (drill 0.8) (layers F.Cu B.Cu) (net 46))
   (segment (start 78.25 164.921292) (end 78.25 152.539219) (width 0.6096) (layer B.Cu) (net 49))
@@
     (polygon
       (pts
-        (xy 15 15) (xy 14.928 95.86) (xy 85.178 95.86) (xy 85.236 138.43) (xy 56.642 138.43)
+        (xy 15 70) (xy 14.928 95.86) (xy 85.178 95.86) (xy 85.236 138.43) (xy 56.642 138.43)
         (xy 56.642 146.05) (xy 53.34 146.05) (xy 53.34 158.496) (xy 50.038 158.496) (xy 50.038 194.564)
-        (xy 169.926 194.564) (xy 170 155) (xy 275 155) (xy 275 15)
+        (xy 164 194.5) (xy 164 155) (xy 164 70)
       )
     )

Commit message: layout changes
Parts:
- moved C23 27.6 mm to (87.8, 164.1), turned to 270 degrees
- moved R19 27.5 mm to (85.0, 164.1), turned to 90 degrees
- moved D8 16.0 mm to (84.0, 158.8), turned to 180 degrees
- moved C22 9.29 mm to (76.8, 164.0), turned to 90 degrees
- moved R18 8.12 mm to (82.2, 164.0), turned to 270 degrees
- moved R17 7.70 mm to (79.5, 164.0), turned to 90 degrees
- moved C20 6.65 mm to (64.4, 163.1), turned to 0 degrees
- moved C11 2.94 mm to (64.4, 160.7)
- moved C12 2.55 mm to (64.4, 158.2)
- moved C15 1.29 mm to (102.6, 162.4)
Routing:
- net /DIGITAL_COMM/ADCH0: track 90.1 -> 52.1 mm
- net /DIGITAL_COMM/ADCH1: track 76.5 -> 38.8 mm
- net Net-(C22-Pad1): track 41.2 -> 32.6 mm
- net /DIGITAL_COMM/ADCH2: track 26.9 -> 19.2 mm
- net Net-(C11-Pad1): track 13.9 -> 10.4 mm
- net /DIGITAL_COMM/ADCH3: track 21.0 -> 23.4 mm
- net GNDREF: track 151.2 -> 148.9 mm
- net /DIGITAL_COMM/TEMPSIO: track 7.66 -> 6.78 mm
- net /DIGITAL_COMM/ADMISO: track 10.2 -> 9.41 mm
- net /DIGITAL_COMM/ADMOSI: track 9.65 -> 8.91 mm
- net Net-(C20-Pad2): track 33.2 -> 33.9 mm
- net /DIGITAL_COMM/TEMPSCK: track 7.08 -> 7.59 mm

Commit message: almost final...
Parts:
- removed P10, P12: CONN_01X01, Mounting_Holes:MountingHole_4-5mm
- removed P7, P8: CONN_01X02, libs:PIN_CONN_0.3Inch
- moved C10 59.4 mm to (24.8, 138.8)
- moved R13 29.8 mm to (34.0, 149.2), turned to 90 degrees
- moved C4 29.2 mm to (112.5, 124.0), turned to 90 degrees
- moved P14 28.8 mm to (78.0, 88.5)
- moved C17 24.2 mm to (122.0, 138.5)
- moved C1 22.7 mm to (112.2, 88.2), turned to 270 degrees
- moved C3 22.6 mm to (122.0, 118.5), turned to 90 degrees
- moved C5 22.2 mm to (101.0, 126.8), turned to 0 degrees
- moved C18 20.5 mm to (112.5, 132.9)
- moved C19 19.8 mm to (101.0, 139.8), turned to 0 degrees
- moved D1 18.1 mm to (94.8, 91.2)
- moved U9 17.8 mm to (97.2, 134.8)
- moved C2 17.6 mm to (93.9, 115.8)
- moved U1 17.6 mm to (92.0, 121.8)
- moved U8 17.6 mm to (92.0, 134.7)
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Connections:
- C23 pad 1: /DIGITAL_COMM/ADCH2 -> /DIGITAL_COMM/ADCH3
- D8 pad 1: /DIGITAL_COMM/ADCH2 -> /DIGITAL_COMM/ADCH3
- D8 pad 2: /DIGITAL_COMM/ADCH3 -> /DIGITAL_COMM/ADCH2
- R17 pad 2: /DIGITAL_COMM/ADCH3 -> /DIGITAL_COMM/ADCH2
- R18 pad 1: /DIGITAL_COMM/ADCH3 -> /DIGITAL_COMM/ADCH2
- R19 pad 2: /DIGITAL_COMM/ADCH2 -> /DIGITAL_COMM/ADCH3
Routing:
- net +5V: track 212.5 -> 152.4 mm, vias 3 -> 2
- net +3V3: track 278.9 -> 224.0 mm
- net GNDREF: track 148.9 -> 105.4 mm, vias 7 -> 3
- net AC+: track 234.4 -> 191.2 mm
- net Net-(P14-Pad1): track 19.8 -> 44.1 mm
- net 230VPHASE: track 153.5 -> 131.4 mm
- net Net-(P7-Pad1): track 25.5 -> 7.62 mm, vias 1 -> 0
- net /SSR_N_SENSING/!FAULT: track 52.7 -> 42.3 mm
- net Net-(D6-Pad2): track 12.1 -> 22.2 mm
- net /SSR_N_SENSING/SSR_ON: track 35.1 -> 26.0 mm
- net /DIGITAL_COMM/ADCH2: track 19.2 -> 25.9 mm
- net MOTOR+: track 21.4 -> 14.8 mm
- net 230VNULL: track 73.9 -> 79.8 mm
- net RECT_VCC: track 183.7 -> 177.9 mm
- net AC-: track 210.8 -> 205.4 mm
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
Commit message: final?
Parts:
- R13: footprint Resistors_ThroughHole:Resistor_Horizontal_RM25mm -> Resistors_ThroughHole:Resistor_Horizontal_RM10mm
- moved C1 10.0 mm to (115.5, 97.8)
- moved D1 10.0 mm to (98.0, 100.8)
- moved P14 10.0 mm to (81.2, 98.0)
- moved T1 9.64 mm to (42.4, 114.0)
- moved R13 3.18 mm to (36.2, 147.0), turned to 0 degrees
Routing:
- net 230VPHASE: track 131.4 -> 104.9 mm
- net 230VNULL: track 79.8 -> 67.4 mm
- net Net-(P7-Pad2): track 24.2 -> 15.1 mm
- net Net-(C10-Pad2): track 9.25 -> 17.4 mm
- net RECT_VCC: track 177.9 -> 171.6 mm
- net AC+: track 191.2 -> 185.0 mm
- net Net-(P14-Pad1): track 44.1 -> 47.5 mm
- net AC-: track 205.4 -> 208.2 mm
- net MOTOR+: track 14.8 -> 14.3 mm

Commit message: printed version
Parts:
- added P15: FUSE, Fuse_Holders_and_Fuses:Fuseholder_Fuse_TR5_Littlefuse-No560_No460, F.Cu at (80.0, 107.4)
- moved C13 1.03 mm to (59.0, 148.2)
- moved D7 0.56 mm to (69.0, 157.5)
Routing:
- net AC+: track 185.0 -> 195.5 mm
- net GNDREF: track 105.4 -> 95.3 mm
- net Net-(P14-Pad1): track 47.5 -> 56.9 mm
- net Net-(R8-Pad1): track 26.4 -> 30.2 mm
- net AC-: track 208.2 -> 211.3 mm
- net (no net): track 0.00 -> 2.75 mm
- net Net-(D6-Pad1): track 27.6 -> 29.3 mm
- net Net-(D6-Pad2): track 22.2 -> 23.9 mm
- net RECT_VCC: track 171.6 -> 170.1 mm
- net /DIGITAL_COMM/ADCH1: track 36.1 -> 34.6 mm
- net /SSR_N_SENSING/FAULT_EN: track 46.9 -> 48.3 mm
- net +3V3: track 224.0 -> 224.9 mm

Commit message: save
Parts:
- C11, C12, C21: value C -> 1nF
- C13, C14, C15, C16, C20, C23: value C -> 10uF
- C22: value C -> 0
- R14: value R -> 150
- R15: value R -> 1k
- R16, R19: value R -> 100k
- R17: value R -> 2k
- R18: value R -> 3k
Connections:
- P11 pad 1: Net-(P11-Pad1) -> (no net)
- P13 pad 1: Net-(P13-Pad1) -> (no net)
- P2 pad 1: Net-(P2-Pad1) -> (no net)
- P2 pad 10: Net-(P2-Pad10) -> (no net)
- P2 pad 12: Net-(P2-Pad12) -> (no net)
- P2 pad 13: Net-(P2-Pad13) -> (no net)
- P2 pad 14: Net-(P2-Pad14) -> (no net)
- P2 pad 16: Net-(P2-Pad16) -> (no net)
- P2 pad 18: Net-(P2-Pad18) -> (no net)
- P2 pad 19: Net-(P2-Pad19) -> (no net)
- P2 pad 20: Net-(P2-Pad20) -> (no net)
- P2 pad 22: Net-(P2-Pad22) -> (no net)
- P2 pad 24: Net-(P2-Pad24) -> (no net)
- P2 pad 26: Net-(P2-Pad26) -> (no net)
- P2 pad 28: Net-(P2-Pad28) -> (no net)
- P2 pad 3: Net-(P2-Pad3) -> (no net)
- P2 pad 30: Net-(P2-Pad30) -> (no net)
- P2 pad 32: Net-(P2-Pad32) -> (no net)
- P2 pad 34: Net-(P2-Pad34) -> (no net)
- P2 pad 36: Net-(P2-Pad36) -> (no net)
- P2 pad 37: Net-(P2-Pad37) -> (no net)
- P2 pad 38: Net-(P2-Pad38) -> (no net)
- P2 pad 39: Net-(P2-Pad39) -> (no net)
- P2 pad 4: Net-(P2-Pad4) -> (no net)
- P2 pad 6: Net-(P2-Pad6) -> (no net)
- P2 pad 8: Net-(P2-Pad8) -> (no net)
- U5 pad 5: Net-(U5-Pad5) -> (no net)
- U5 pad 6: Net-(U5-Pad6) -> (no net)
- U6 pad 3: Net-(U6-Pad3) -> (no net)
- U6 pad 5: Net-(U6-Pad5) -> (no net)
- U6 pad 6: Net-(U6-Pad6) -> (no net)
Routing:
- net /DIGITAL_COMM/ADCH1: track 34.6 -> 37.4 mm
- net (no net): track 2.75 -> 0.00 mm
Other:
- board text added: "hiba!!! GND"
- board text added: "hibák: 1., DIY nyák táp pol C-knél 2., DIY nyák diode bridge-nél 3.,40-es csatlakozó mérete nagyobb 4., sorkapcsok mérete nagyobb 5., DIY nyák 40-es csatlakozó előtti via"
