File: PWR_module.sch (KiCad schematic (older format))
At the start: 13 parts

Commit message: sch almost ready
Parts:
- removed C? (x2): C, symbol C
- removed C?: CP, symbol CP
- removed P?: CONN_01X02, symbol CONN_01X02
- removed U?: LM7808CT, TO-220, symbol LM7808CT
- added C17, C19: C, Capacitors_SMD:C_1206_HandSoldering, symbol C
- added C18: CP, Capacitors_Elko_ThroughHole:Elko_vert_31.5x16mm_RM7.5, symbol CP
- added U7: ua78m33, Transistors_TO-220:TO-220_Neutral123_Vertical_LargePads, symbol 7805
- added U8: 7805, Transistors_TO-220:TO-220_Neutral123_Vertical_LargePads, symbol 7805
- added U9: SPX2920M3-3.3, libs:SOT223-ti-pin2is4too, symbol SPX2920M3-3.3
- C1, C4: renamed from C?; footprint (none) -> Capacitors_Elko_ThroughHole:Elko_vert_31.5x16mm_RM7.5
- C2, C3, C5: renamed from C?; footprint (none) -> Capacitors_SMD:C_1206_HandSoldering
- D1: renamed from D?; footprint (none) -> libs:rb1a_mb6sbridge
- T1: renamed from T?; footprint (none) -> libs:MYRRA_44266
- U1: renamed from U?; footprint SOT223 -> libs:SOT223-ti-pin2is4too
Connections:
- net labels added: +3.3V, +5V, RECT_VCC
- net labels removed: 3.3V, 8V, GND
- wire segments 26 -> 24

Commit message: sch ready, begining of layout
Parts:
- removed U7: ua78m33, Transistors_TO-220:TO-220_Neutral123_Vertical_LargePads, symbol 7805
- removed U8: 7805, Transistors_TO-220:TO-220_Neutral123_Vertical_LargePads, symbol 7805
- added U7: SPX2920M3-3.3, libs:SOT223-ti-pin2is4too, symbol SPX2920M3-3.3
- added U8: SPX2920M3-3.3, Transistors_TO-220:TO-220_Neutral123_Vertical_LargePads, symbol SPX2920M3-3.3
- U1: footprint libs:SOT223-ti-pin2is4too -> Transistors_TO-220:TO-220_Neutral123_Vertical_LargePads
Other:
- moved on the sheet: U1
Changed lines of the file:
@@
 	6050 2850 6900 2850
 Connection ~ 6400 2850
-$Comp
-L SPX2920M3-3.3 U1
-U 1 1 5614DDD0
-P 7300 2900
-F 0 "U1" H 7300 3150 40  0000 C CNN
-F 1 "SPX2920M3-3.3" H 7300 3100 40  0000 C CNN
-F 2 "libs:SOT223-ti-pin2is4too" H 7300 3000 35  0000 C CIN
-F 3 "" H 7300 2900 60  0000 C CNN
-	1    7300 2900
-	1    0    0    -1
-$EndComp
 Wire Wire Line
 	7300 3850 7300 3150
@@
 Connection ~ 7800 3850
 $Comp
-L GNDREF #PWR07
+L GNDREF #PWR010
 U 1 1 5614E0AD
 P 6850 3850
-F 0 "#PWR07" H 6850 3600 50  0001 C CNN
+F 0 "#PWR010" H 6850 3600 50  0001 C CNN
 F 1 "GNDREF" H 6850 3700 50  0000 C CNN
 F 2 "" H 6850 3850 60  0000 C CNN
@@
 	4650 3850 8200 3850
 $Comp
-L +3.3V #PWR08
+L +3.3V #PWR011
 U 1 1 561BB1C6
 P 8000 2850
-F 0 "#PWR08" H 8000 2700 50  0001 C CNN
+F 0 "#PWR011" H 8000 2700 50  0001 C CNN
 F 1 "+3.3V" H 8000 2990 50  0000 C CNN
 F 2 "" H 8000 2850 60  0000 C CNN
@@
 Text GLabel 6400 2850 1    60   Input ~ 0
 RECT_VCC
-$Comp
-L 7805 U8
-U 1 1 56259002
-P 7400 4250
-F 0 "U8" H 7550 4054 60  0000 C CNN
-F 1 "7805" H 7400 4450 60  0000 C CNN
-F 2 "Transistors_TO-220:TO-220_Neutral123_Vertical_LargePads" H 7400 4250 60  0001 C CNN
-F 3 "" H 7400 4250 60  0000 C CNN
-	1    7400 4250
-	1    0    0    -1
-$EndComp
-$Comp
-L 7805 U7
-U 1 1 5625904F
-P 7300 2150
-F 0 "U7" H 7450 1954 60  0000 C CNN
-F 1 "ua78m33" H 7300 2350 60  0000 C CNN
-F 2 "Transistors_TO-220:TO-220_Neutral123_Vertical_LargePads" H 7300 2150 60  0001 C CNN
-F 3 "" H 7300 2150 60  0000 C CNN
-	1    7300 2150
-	1    0    0    -1
-$EndComp
 Wire Wire Line
 	6900 2850 6900 2100
@@
 Connection ~ 7900 2850
 $Comp
-L GNDREF #PWR09
+L GNDREF #PWR012
 U 1 1 56259110
 P 7300 2400
-F 0 "#PWR09" H 7300 2150 50  0001 C CNN
+F 0 "#PWR012" H 7300 2150 50  0001 C CNN
 F 1 "GNDREF" H 7300 2250 50  0000 C CNN
 F 2 "" H 7300 2400 60  0000 C CNN
@@
 Connection ~ 6950 3850
 $Comp
-L GNDREF #PWR010
+L GNDREF #PWR013
 U 1 1 562593C0
 P 7400 4500
-F 0 "#PWR010" H 7400 4250 50  0001 C CNN
+F 0 "#PWR013" H 7400 4250 50  0001 C CNN
 F 1 "GNDREF" H 7400 4350 50  0000 C CNN
 F 2 "" H 7400 4500 60  0000 C CNN
@@
 Connection ~ 8100 4500
 $Comp
-L GNDREF #PWR011
+L GNDREF #PWR014
 U 1 1 5625976C
 P 8100 4500
-F 0 "#PWR011" H 8100 4250 50  0001 C CNN
+F 0 "#PWR014" H 8100 4250 50  0001 C CNN
 F 1 "GNDREF" H 8100 4350 50  0000 C CNN
 F 2 "" H 8100 4500 60  0000 C CNN
@@
 $EndComp
 $Comp
-L +5V #PWR012
+L +5V #PWR015
 U 1 1 56259809
 P 8300 4200
-F 0 "#PWR012" H 8300 4050 50  0001 C CNN
+F 0 "#PWR015" H 8300 4050 50  0001 C CNN
 F 1 "+5V" H 8300 4340 50  0000 C CNN
 F 2 "" H 8300 4200 60  0000 C CNN
@@
 Connection ~ 6950 4200
 $Comp
-L +5V #PWR013
+L +5V #PWR016
 U 1 1 56259AAC
 P 7850 4900
-F 0 "#PWR013" H 7850 4750 50  0001 C CNN
+F 0 "#PWR016" H 7850 4750 50  0001 C CNN
 F 1 "+5V" H 7850 5040 50  0000 C CNN
 F 2 "" H 7850 4900 60  0000 C CNN
@@
 $EndComp
 $Comp
-L GNDREF #PWR014
+L GNDREF #PWR017
 U 1 1 56259AE1
 P 7450 5200
-F 0 "#PWR014" H 7450 4950 50  0001 C CNN
+F 0 "#PWR017" H 7450 4950 50  0001 C CNN
 F 1 "GNDREF" H 7450 5050 50  0000 C CNN
 F 2 "" H 7450 5200 60  0000 C CNN
@@
 	1    0    0    -1
 $EndComp
+$Comp
+L SPX2920M3-3.3 U1
+U 1 1 5614DDD0
+P 7300 2150
+F 0 "U1" H 7300 2400 40  0000 C CNN
+F 1 "SPX2920M3-3.3" H 7300 2350 40  0000 C CNN
+F 2 "Transistors_TO-220:TO-220_Neutral123_Vertical_LargePads" H 7300 2250 35  0000 C CIN
+F 3 "" H 7300 2150 60  0000 C CNN
+	1    7300 2150
+	1    0    0    -1
+$EndComp
+$Comp
+L SPX2920M3-3.3 U7
+U 1 1 5627402E
+P 7300 2900
+F 0 "U7" H 7300 3150 40  0000 C CNN
+F 1 "SPX2920M3-3.3" H 7300 3100 40  0000 C CNN
+F 2 "libs:SOT223-ti-pin2is4too" H 7300 3000 35  0000 C CIN
+F 3 "" H 7300 2900 60  0000 C CNN
+	1    7300 2900
+	1    0    0    -1
+$EndComp
+$Comp
+L SPX2920M3-3.3 U8
+U 1 1 56274209
+P 7400 4250
+F 0 "U8" H 7400 4500 40  0000 C CNN
+F 1 "SPX2920M3-3.3" H 7400 4450 40  0000 C CNN
+F 2 "Transistors_TO-220:TO-220_Neutral123_Vertical_LargePads" H 7400 4350 35  0000 C CIN
+F 3 "" H 7400 4250 60  0000 C CNN
+	1    7400 4250
+	1    0    0    -1
+$EndComp

Commit message: PWR layout
Connections:
- net labels added: 230VNULL, 230VPHASE
- wire segments 24 -> 25
Changed lines of the file:
@@
 	1    0    0    -1
 $EndComp
-Wire Wire Line
-	2350 3050 2750 3050
-Wire Wire Line
-	2750 2650 2350 2650
-Wire Wire Line
-	3550 2650 3550 2150
-Wire Wire Line
-	3550 2150 5350 2150
-Wire Wire Line
-	5350 3550 3550 3550
-Wire Wire Line
-	3550 3550 3550 3050
-Wire Wire Line
-	4650 2850 4650 3850
-Wire Wire Line
-	6400 3850 6400 3150
-Wire Wire Line
-	6650 3850 6650 3150
-Connection ~ 6400 3850
-Wire Wire Line
-	6050 2850 6900 2850
-Connection ~ 6400 2850
-Wire Wire Line
-	7300 3850 7300 3150
-Connection ~ 6650 3850
-Connection ~ 6650 2850
 $Comp
 L C C3
@@
 	1    0    0    -1
 $EndComp
-Wire Wire Line
-	7700 2850 8200 2850
-Connection ~ 7800 2850
-Connection ~ 8000 2850
-Wire Wire Line
-	8200 3850 8200 3150
-Connection ~ 7300 3850
-Wire Wire Line
-	8000 3850 8000 3150
-Connection ~ 8000 3850
-Wire Wire Line
-	7800 3850 7800 3150
-Connection ~ 7800 3850
 $Comp
 L GNDREF #PWR010
@@
 	1    0    0    -1
 $EndComp
-Connection ~ 8200 3850
-Text GLabel 2350 2650 0    60   Input ~ 0
+Text GLabel 3550 2150 1    60   Input ~ 0
 AC+
-Text GLabel 2350 3050 0    60   Input ~ 0
+Text GLabel 3550 3550 3    60   Input ~ 0
 AC-
-Wire Wire Line
-	4650 3850 8200 3850
 $Comp
 L +3.3V #PWR011
@@
 Text GLabel 6400 2850 1    60   Input ~ 0
 RECT_VCC
-Wire Wire Line
-	6900 2850 6900 2100
-Wire Wire Line
-	7700 2100 7900 2100
-Wire Wire Line
-	7900 2100 7900 2850
-Connection ~ 7900 2850
 $Comp
 L GNDREF #PWR012
@@
 	1    0    0    -1
 $EndComp
-Wire Wire Line
-	6950 3850 6950 4900
-Wire Wire Line
-	6950 4200 7000 4200
-Connection ~ 6950 3850
 $Comp
 L GNDREF #PWR013
@@
 	1    0    0    -1
 $EndComp
-Wire Wire Line
-	7800 4200 8300 4200
-Connection ~ 7900 4200
-Connection ~ 8100 4200
-Wire Wire Line
-	7900 4500 8300 4500
-Connection ~ 8100 4500
 $Comp
 L GNDREF #PWR014
@@
 	1    0    0    -1
 $EndComp
-Wire Wire Line
-	6950 4900 7050 4900
-Connection ~ 6950 4200
 $Comp
 L +5V #PWR016
@@
 	1    0    0    -1
 $EndComp
+Wire Wire Line
+	2350 3050 2750 3050
+Wire Wire Line
+	2750 2650 2350 2650
+Wire Wire Line
+	3550 2650 3550 2150
+Wire Wire Line
+	3550 2150 5350 2150
+Wire Wire Line
+	5350 3550 3550 3550
+Wire Wire Line
+	3550 3550 3550 3050
+Wire Wire Line
+	4650 2850 4650 3850
+Wire Wire Line
+	6400 3850 6400 3150
+Wire Wire Line
+	6650 3850 6650 3150
+Connection ~ 6400 3850
+Wire Wire Line
+	6050 2850 6900 2850
+Connection ~ 6400 2850
+Wire Wire Line
+	7300 3850 7300 3150
+Connection ~ 6650 3850
+Connection ~ 6650 2850
+Wire Wire Line
+	7700 2850 8200 2850
+Connection ~ 7800 2850
+Connection ~ 8000 2850
+Wire Wire Line
+	8200 3850 8200 3150
+Connection ~ 7300 3850
+Wire Wire Line
+	8000 3850 8000 3150
+Connection ~ 8000 3850
+Wire Wire Line
+	7800 3850 7800 3150
+Connection ~ 7800 3850
+Connection ~ 8200 3850
+Wire Wire Line
+	4650 3850 8550 3850
+Wire Wire Line
+	6900 2850 6900 2100
+Wire Wire Line
+	7700 2100 7900 2100
+Wire Wire Line
+	7900 2100 7900 2850
+Connection ~ 7900 2850
+Wire Wire Line
+	6950 4200 6950 4900
+Wire Wire Line
+	6950 4200 7000 4200
+Wire Wire Line
+	7800 4200 8300 4200
+Connection ~ 7900 4200
+Connection ~ 8100 4200
+Wire Wire Line
+	7900 4500 8550 4500
+Connection ~ 8100 4500
+Wire Wire Line
+	6950 4900 7050 4900
+Connection ~ 6950 4200
+Wire Wire Line
+	8550 4500 8550 3850
+Connection ~ 8300 4500
+Text GLabel 6950 4450 0    60   Input ~ 0
+RECT_VCC
+Text GLabel 2350 2650 0    60   Input ~ 0
+230VPHASE
+Text GLabel 2350 3050 0    60   Input ~ 0
+230VNULL
 $EndSCHEMATC

Commit message: maybe final
Parts:
- added P14: CONN_01X02, libs:PIN_CONN_0.3Inch, symbol CONN_01X02
Connections:
- wire segments 25 -> 28

Commit message: printed version
Parts:
- added P15: FUSE, Fuse_Holders_and_Fuses:Fuseholder_Fuse_TR5_Littlefuse-No560_No460, symbol CONN_01X02
Changed lines of the file:
@@
 $EndComp
 Wire Wire Line
-	4750 2150 4750 2050
+	4750 2050 4750 2250
 Connection ~ 4750 2150
 Wire Wire Line
-	4850 2050 4850 2150
+	4850 2050 4850 2250
 Connection ~ 4850 2150
 Wire Wire Line
@@
 Wire Wire Line
 	3550 2150 4750 2150
+$Comp
+L CONN_01X02 P15
+U 1 1 5634C69D
+P 4800 2450
+F 0 "P15" H 4800 2600 50  0000 C CNN
+F 1 "FUSE" V 4900 2450 50  0000 C CNN
+F 2 "Fuse_Holders_and_Fuses:Fuseholder_Fuse_TR5_Littlefuse-No560_No460" H 4800 2450 60  0000 C CNN
+F 3 "" H 4800 2450 60  0000 C CNN
+	1    4800 2450
+	0    1    1    0
+$EndComp
 $EndSCHEMATC

Commit message: save
Parts:
- D1: symbol Diode_Bridge -> Diode_Bridge-RESCUE-viztisztito
Changed lines of the file:
@@
 EESchema Schematic File Version 2
+LIBS:viztisztito-rescue
 LIBS:power
 LIBS:device
@@
 	6050 2850 6900 2850
 $Comp
-L Diode_Bridge D1
+L Diode_Bridge-RESCUE-viztisztito D1
 U 1 1 5614DBFC
 P 5350 2850
