File: water_level.sch (KiCad schematic (older format))
At the start: 22 parts

Commit message: sch almost ready
Parts:
- removed P?: CONN_01X06, symbol CONN_01X06
- C6, C7, C8, C9: renamed from C?; footprint (none) -> Capacitors_SMD:C_1206_HandSoldering
- D2, D3, D4, D5: renamed from D?; footprint (none) -> libs:MB6S_SMD
- R1, R10, R11, R12, R2, R3, R4, R5, R6, R7, R8, R9: renamed from R?; footprint (none) -> Resistors_SMD:R_1206_HandSoldering
- U2: renamed from U?; footprint DIP-16 -> Housings_SOIC:SOIC-16_3.9x9.9mm_Pitch1.27mm
Connections:
- net labels added: WL0, WL1, WL2, WL3
- net labels removed: 3.3V, AC+, GND
- wire segments 55 -> 51

Commit message: save
Parts:
- D2, D3, D4, D5: symbol Diode_Bridge -> Diode_Bridge-RESCUE-viztisztito
Connections:
- net labels added: GND1, GND2, GND3, GND4
Changed lines of the file:
@@
 EESchema Schematic File Version 2
+LIBS:viztisztito-rescue
 LIBS:power
 LIBS:device
@@
 $EndDescr
 $Comp
-L Diode_Bridge D2
+L Diode_Bridge-RESCUE-viztisztito D2
 U 1 1 5614FA35
 P 1850 1700
+AR Path="/5614FA35" Ref="D2"  Part="1"
+AR Path="/5614D8B0/5614FA35" Ref="D2"  Part="1"
 F 0 "D2" H 1850 1750 50  0000 C CNN
 F 1 "Diode_Bridge" H 1850 1650 50  0000 C CNN
@@
 $EndComp
 $Comp
-L Diode_Bridge D3
+L Diode_Bridge-RESCUE-viztisztito D3
 U 1 1 5614FABD
 P 1850 3400
+AR Path="/5614FABD" Ref="D3"  Part="1"
+AR Path="/5614D8B0/5614FABD" Ref="D3"  Part="1"
 F 0 "D3" H 1850 3450 50  0000 C CNN
 F 1 "Diode_Bridge" H 1850 3350 50  0000 C CNN
@@
 $EndComp
 $Comp
-L Diode_Bridge D5
+L Diode_Bridge-RESCUE-viztisztito D5
 U 1 1 5614FAED
 P 1900 5100
+AR Path="/5614FAED" Ref="D5"  Part="1"
+AR Path="/5614D8B0/5614FAED" Ref="D5"  Part="1"
 F 0 "D5" H 1900 5150 50  0000 C CNN
 F 1 "Diode_Bridge" H 1900 5050 50  0000 C CNN
@@
 $EndComp
 $Comp
-L Diode_Bridge D4
+L Diode_Bridge-RESCUE-viztisztito D4
 U 1 1 5614FB32
 P 1850 6750
+AR Path="/5614FB32" Ref="D4"  Part="1"
+AR Path="/5614D8B0/5614FB32" Ref="D4"  Part="1"
 F 0 "D4" H 1850 6800 50  0000 C CNN
 F 1 "Diode_Bridge" H 1850 6700 50  0000 C CNN
@@
 Text GLabel 1850 7450 0    60   Input ~ 0
 AC-
-$Comp
-L GNDREF #PWR018
-U 1 1 56150471
-P 1150 1700
-F 0 "#PWR018" H 1150 1450 50  0001 C CNN
-F 1 "GNDREF" H 1150 1550 50  0000 C CNN
-F 2 "" H 1150 1700 60  0000 C CNN
-F 3 "" H 1150 1700 60  0000 C CNN
-	1    1150 1700
-	0    1    1    0
-$EndComp
-$Comp
-L GNDREF #PWR019
-U 1 1 56150528
-P 1150 3400
-F 0 "#PWR019" H 1150 3150 50  0001 C CNN
-F 1 "GNDREF" H 1150 3250 50  0000 C CNN
-F 2 "" H 1150 3400 60  0000 C CNN
-F 3 "" H 1150 3400 60  0000 C CNN
-	1    1150 3400
-	0    1    1    0
-$EndComp
-$Comp
-L GNDREF #PWR020
-U 1 1 56150628
-P 1200 5100
-F 0 "#PWR020" H 1200 4850 50  0001 C CNN
-F 1 "GNDREF" H 1200 4950 50  0000 C CNN
-F 2 "" H 1200 5100 60  0000 C CNN
-F 3 "" H 1200 5100 60  0000 C CNN
-	1    1200 5100
-	0    1    1    0
-$EndComp
-$Comp
-L GNDREF #PWR021
-U 1 1 56150741
-P 1150 6750
-F 0 "#PWR021" H 1150 6500 50  0001 C CNN
-F 1 "GNDREF" H 1150 6600 50  0000 C CNN
-F 2 "" H 1150 6750 60  0000 C CNN
-F 3 "" H 1150 6750 60  0000 C CNN
-	1    1150 6750
-	0    1    1    0
-$EndComp
 $Comp
 L LTV-847 U2
@@
 	1    3050 6900
 	-1   0    0    1
-$EndComp
-$Comp
-L GNDREF #PWR022
-U 1 1 56151F2F
-P 3050 2050
-F 0 "#PWR022" H 3050 1800 50  0001 C CNN
-F 1 "GNDREF" H 3050 1900 50  0000 C CNN
-F 2 "" H 3050 2050 60  0000 C CNN
-F 3 "" H 3050 2050 60  0000 C CNN
-	1    3050 2050
-	1    0    0    -1
-$EndComp
-$Comp
-L GNDREF #PWR023
-U 1 1 56151F93
-P 3000 3800
-F 0 "#PWR023" H 3000 3550 50  0001 C CNN
-F 1 "GNDREF" H 3000 3650 50  0000 C CNN
-F 2 "" H 3000 3800 60  0000 C CNN
-F 3 "" H 3000 3800 60  0000 C CNN
-	1    3000 3800
-	1    0    0    -1
-$EndComp
-$Comp
-L GNDREF #PWR024
-U 1 1 561522AC
-P 3000 5500
-F 0 "#PWR024" H 3000 5250 50  0001 C CNN
-F 1 "GNDREF" H 3000 5350 50  0000 C CNN
-F 2 "" H 3000 5500 60  0000 C CNN
-F 3 "" H 3000 5500 60  0000 C CNN
-	1    3000 5500
-	1    0    0    -1
-$EndComp
-$Comp
-L GNDREF #PWR025
-U 1 1 56152537
-P 2950 7150
-F 0 "#PWR025" H 2950 6900 50  0001 C CNN
-F 1 "GNDREF" H 2950 7000 50  0000 C CNN
-F 2 "" H 2950 7150 60  0000 C CNN
-F 3 "" H 2950 7150 60  0000 C CNN
-	1    2950 7150
-	1    0    0    -1
-$EndComp
-$Comp
-L GNDREF #PWR026
-U 1 1 561527C4
-P 3850 3650
-F 0 "#PWR026" H 3850 3400 50  0001 C CNN
-F 1 "GNDREF" H 3850 3500 50  0000 C CNN
-F 2 "" H 3850 3650 60  0000 C CNN
-F 3 "" H 3850 3650 60  0000 C CNN
-	1    3850 3650
-	0    1    1    0
-$EndComp
-$Comp
-L GNDREF #PWR027
-U 1 1 56152B89
-P 3850 3350
-F 0 "#PWR027" H 3850 3100 50  0001 C CNN
-F 1 "GNDREF" H 3850 3200 50  0000 C CNN
-F 2 "" H 3850 3350 60  0000 C CNN
-F 3 "" H 3850 3350 60  0000 C CNN
-	1    3850 3350
-	0    1    1    0
-$EndComp
-$Comp
-L GNDREF #PWR028
-U 1 1 56152F36
-P 3850 3050
-F 0 "#PWR028" H 3850 2800 50  0001 C CNN
-F 1 "GNDREF" H 3850 2900 50  0000 C CNN
-F 2 "" H 3850 3050 60  0000 C CNN
-F 3 "" H 3850 3050 60  0000 C CNN
-	1    3850 3050
-	0    1    1    0
-$EndComp
-$Comp
-L GNDREF #PWR029
-U 1 1 561530F1
-P 3850 2750
-F 0 "#PWR029" H 3850 2500 50  0001 C CNN
-F 1 "GNDREF" H 3850 2600 50  0000 C CNN
-F 2 "" H 3850 2750 60  0000 C CNN
-F 3 "" H 3850 2750 60  0000 C CNN
-	1    3850 2750
-	0    1    1    0
 $EndComp
 Connection ~ 3050 6750
@@
 Wire Wire Line
 	750  4250 1350 4250
+Text Label 3850 2750 2    60   ~ 0
+GND1
+Text Label 3050 2050 3    60   ~ 0
+GND1
+Text Label 1150 1700 3    60   ~ 0
+GND1
+Text Label 3850 3050 2    60   ~ 0
+GND2
+Text Label 3850 3350 2    60   ~ 0
+GND3
+Text Label 3850 3650 2    60   ~ 0
+GND4
+Text Label 3000 3800 3    60   ~ 0
+GND2
+Text Label 1150 3400 3    60   ~ 0
+GND2
+Text Label 3000 5500 3    60   ~ 0
+GND3
+Text Label 1200 5100 3    60   ~ 0
+GND3
+Text Label 2950 7150 3    60   ~ 0
+GND4
+Text Label 1150 6750 3    60   ~ 0
+GND4
 $EndSCHEMATC
