File: viztisztito.sch (KiCad schematic (older format))
At the start: 3 parts, among them P1 BOARD_CONN

Commit message: before new pcb; - the order of the gpio pins have changed in accordance with olinuxino - indicator leds have been added for debugging - ad current pin added for debugging
Parts:
- added D1, D2, D3, D4, D5, D6, D7, D8: LED, LEDs:LED_1206, symbol LED
- added R1, R2, R3: 330, Resistors_SMD:R_1206_HandSoldering, symbol R
- added R4, R5, R6, R7, R8: 1k, Resistors_SMD:R_1206_HandSoldering, symbol R
Connections:
- wire segments 31 -> 57
Other:
- note added: "Indicator LEDs"
- note removed: "MEGFORDÍTOTT SORREND!"

Commit message: unconnect the 3.3V pin from olinuxino (it has an own dc-dc converter)
Connections:
- net labels removed: +3.3V
Changed lines of the file:
@@
 Text GLabel 7900 4600 1    60   Input ~ 0
 +5V
-Text GLabel 7900 5400 3    60   Input ~ 0
-+3.3V
 $Comp
 L R R2

Commit message: changes towards the liteSOM drive.
Parts:
- R1, R2, R3: value 330 -> 2k
- R4, R5, R6, R7, R8: value 1k -> 2k
Connections:
- net labels added: +3.3V
- wire segments 57 -> 56
Changed lines of the file:
@@
 LIBS:vtx-214-015-112
 LIBS:viztisztito-cache
+LIBS:dc-dc
+LIBS:cmos_ieee
+LIBS:zetex
+LIBS:RFSolutions
 EELAYER 25 0
 EELAYER END
 $Descr A4 11693 8268
 encoding utf-8
-Sheet 1 5
+Sheet 1 6
 Title ""
 Date ""
@@
 	8900 5100 8900 5400
 Wire Wire Line
-	8800 5100 8800 5400
-Wire Wire Line
 	8700 5100 8700 5400
 Wire Wire Line
@@
 	8400 5100 8400 5400
 Wire Wire Line
+	8300 5100 8300 5400
+Wire Wire Line
 	8100 5100 8100 5400
 Wire Wire Line
 	8000 5100 8000 5400
-Wire Wire Line
-	7900 5100 7900 5400
 Wire Wire Line
 	8000 4600 8000 4250
@@
 Text Label 8250 1850 0    60   ~ 0
 AD_CLK
-Text Label 8300 4250 1    60   ~ 0
+Text Label 8300 4150 1    60   ~ 0
 DWL0
-Text Label 8200 4250 1    60   ~ 0
+Text Label 8200 4150 1    60   ~ 0
 DWL1
-Text Label 8100 4250 1    60   ~ 0
+Text Label 8100 4150 1    60   ~ 0
 DWL2
-Text Label 8000 4250 1    60   ~ 0
+Text Label 8000 4150 1    60   ~ 0
 DWL3
 Text Label 9300 4250 1    60   ~ 0
@@
 P 9850 3900
 F 0 "R2" V 9930 3900 50  0000 C CNN
-F 1 "330" V 9850 3900 50  0000 C CNN
+F 1 "2k" V 9850 3900 50  0000 C CNN
 F 2 "Resistors_SMD:R_1206_HandSoldering" V 9780 3900 50  0001 C CNN
 F 3 "http://hu.farnell.com/multicomp/mcwr12x3300ftl/res-thick-film-330r-1-0-25w-1206/dp/2447504" H 9850 3900 50  0001 C CNN
@@
 P 9500 3900
 F 0 "R1" V 9580 3900 50  0000 C CNN
-F 1 "330" V 9500 3900 50  0000 C CNN
+F 1 "2k" V 9500 3900 50  0000 C CNN
 F 2 "Resistors_SMD:R_1206_HandSoldering" V 9430 3900 50  0001 C CNN
 F 3 "http://hu.farnell.com/multicomp/mcwr12x3300ftl/res-thick-film-330r-1-0-25w-1206/dp/2447504" H 9500 3900 50  0001 C CNN
@@
 P 10200 3900
 F 0 "R3" V 10280 3900 50  0000 C CNN
-F 1 "330" V 10200 3900 50  0000 C CNN
+F 1 "2k" V 10200 3900 50  0000 C CNN
 F 2 "Resistors_SMD:R_1206_HandSoldering" V 10130 3900 50  0001 C CNN
 F 3 "http://hu.farnell.com/multicomp/mcwr12x3300ftl/res-thick-film-330r-1-0-25w-1206/dp/2447504" H 10200 3900 50  0001 C CNN
@@
 P 5600 3950
 F 0 "R4" V 5680 3950 50  0000 C CNN
-F 1 "1k" V 5600 3950 50  0000 C CNN
+F 1 "2k" V 5600 3950 50  0000 C CNN
 F 2 "Resistors_SMD:R_1206_HandSoldering" V 5530 3950 50  0001 C CNN
 F 3 "http://hu.farnell.com/multicomp/mcwr12x1001ftl/res-thick-film-1k-1-0-25w-1206/dp/2447473" H 5600 3950 50  0001 C CNN
@@
 P 5900 3950
 F 0 "R5" V 5980 3950 50  0000 C CNN
-F 1 "1k" V 5900 3950 50  0000 C CNN
+F 1 "2k" V 5900 3950 50  0000 C CNN
 F 2 "Resistors_SMD:R_1206_HandSoldering" V 5830 3950 50  0001 C CNN
 F 3 "http://hu.farnell.com/multicomp/mcwr12x1001ftl/res-thick-film-1k-1-0-25w-1206/dp/2447473" H 5900 3950 50  0001 C CNN
@@
 P 6200 3950
 F 0 "R6" V 6280 3950 50  0000 C CNN
-F 1 "1k" V 6200 3950 50  0000 C CNN
+F 1 "2k" V 6200 3950 50  0000 C CNN
 F 2 "Resistors_SMD:R_1206_HandSoldering" V 6130 3950 50  0001 C CNN
 F 3 "http://hu.farnell.com/multicomp/mcwr12x1001ftl/res-thick-film-1k-1-0-25w-1206/dp/2447473" H 6200 3950 50  0001 C CNN
@@
 P 6500 3950
 F 0 "R7" V 6580 3950 50  0000 C CNN
-F 1 "1k" V 6500 3950 50  0000 C CNN
+F 1 "2k" V 6500 3950 50  0000 C CNN
 F 2 "Resistors_SMD:R_1206_HandSoldering" V 6430 3950 50  0001 C CNN
 F 3 "http://hu.farnell.com/multicomp/mcwr12x1001ftl/res-thick-film-1k-1-0-25w-1206/dp/2447473" H 6500 3950 50  0001 C CNN
@@
 P 6800 3950
 F 0 "R8" V 6880 3950 50  0000 C CNN
-F 1 "1k" V 6800 3950 50  0000 C CNN
+F 1 "2k" V 6800 3950 50  0000 C CNN
 F 2 "Resistors_SMD:R_1206_HandSoldering" V 6730 3950 50  0001 C CNN
 F 3 "http://hu.farnell.com/multicomp/mcwr12x1001ftl/res-thick-film-1k-1-0-25w-1206/dp/2447473" H 6800 3950 50  0001 C CNN
@@
 Text Label 6800 4300 3    60   ~ 0
 DWL0
+Text Label 8300 5400 3    60   ~ 0
+DWL3
+Text Label 8400 5400 3    60   ~ 0
+DWL2
+Text Label 8500 5400 3    60   ~ 0
+DWL1
+Text Label 8600 5400 3    60   ~ 0
+DWL0
+Text GLabel 7900 5700 3    60   Input ~ 0
++3.3V
+$Sheet
+S 1300 1000 1550 1150
+U 599A5341
+F0 "system_on_module" 60
+F1 "system_on_module.sch" 60
+$EndSheet
 $EndSCHEMATC

Commit message: this version contains all the important modules: - wifi - sd-card - usb-debug - litesom - gpio connections it does NOT contain the power module and the revision of the voltages
Parts:
- removed P1: BOARD_CONN, water:olinuxino_im233_ver2, symbol CONN_02X20
Connections:
- net labels added: INDICATOR_LED_0, INDICATOR_LED_1, INDICATOR_LED_2
- net labels removed: +3.3V, +5V
- wire segments 56 -> 30
Other:
- note removed: "Embedded Control Computer"
Changed lines of the file:
@@
 LIBS:zetex
 LIBS:RFSolutions
+LIBS:switches
 EELAYER 25 0
 EELAYER END
 $Descr A4 11693 8268
 encoding utf-8
-Sheet 1 6
+Sheet 1 10
 Title ""
 Date ""
@@
 $EndDescr
 $Sheet
-S 1850 6900 1200 950
+S 4750 6350 1200 950
 U 5614D811
 F0 "PWR_module" 60
@@
 $EndSheet
 $Sheet
-S 1250 2500 1200 950
+S 1250 3800 1200 950
 U 5614D8B0
 F0 "water_level" 60
 F1 "water_level.sch" 60
-F2 "water_level_0" O R 2450 2600 60
-F3 "water_level_1" O R 2450 2700 60
-F4 "water_level_2" O R 2450 2800 60
-F5 "water_level_3" O R 2450 2900 60
+F2 "water_level_0" O R 2450 3900 60
+F3 "water_level_1" O R 2450 4000 60
+F4 "water_level_2" O R 2450 4100 60
+F5 "water_level_3" O R 2450 4200 60
 $EndSheet
 $Sheet
@@
 F10 "ADCH1" I L 7050 1050 60
 $EndSheet
-$Comp
-L CONN_02X20 P1
-U 1 1 561C12E9
-P 8750 4850
-F 0 "P1" H 8750 5900 50  0000 C CNN
-F 1 "BOARD_CONN" V 8750 4850 50  0000 C CNN
-F 2 "water:olinuxino_im233_ver2" H 8750 3900 60  0001 C CNN
-F 3 "http://hu.farnell.com/wurth-elektronik/61304021021/header-2-54mm-pin-tht-r-a-40way/dp/2356207" H 8750 3900 60  0001 C CNN
-F 4 "http://hu.farnell.com/3m/d89140-0031hk/connector-rcpt-40pos-2row-2-54mm/dp/2672516" H 8750 4850 60  0001 C CNN "idc connector"
-F 5 "http://hu.farnell.com/pro-power/r2651dtsy40sc85/ribbon-cable-40-core-28awg-per/dp/2628367" H 8750 4850 60  0001 C CNN "ribbon cable"
-	1    8750 4850
-	0    1    1    0
-$EndComp
-Wire Wire Line
-	9200 5100 9200 5400
-Wire Wire Line
-	9100 5100 9100 5400
-Wire Wire Line
-	9000 5100 9000 5400
-Wire Wire Line
-	8900 5100 8900 5400
-Wire Wire Line
-	8700 5100 8700 5400
-Wire Wire Line
-	8600 5100 8600 5400
-Wire Wire Line
-	8500 5100 8500 5400
-Wire Wire Line
-	8400 5100 8400 5400
-Wire Wire Line
-	8300 5100 8300 5400
-Wire Wire Line
-	8100 5100 8100 5400
-Wire Wire Line
-	8000 5100 8000 5400
-Wire Wire Line
-	8000 4600 8000 4250
-Wire Wire Line
-	8100 4600 8100 4250
-Wire Wire Line
-	8200 4600 8200 4250
-Wire Wire Line
-	8300 4600 8300 4250
-Wire Wire Line
-	8500 4600 8500 4250
-Wire Wire Line
-	8600 4600 8600 4250
-Wire Wire Line
-	8900 4600 8900 4250
-Wire Wire Line
-	9000 4600 9000 4250
-Wire Wire Line
-	9200 4600 9200 4250
-Wire Wire Line
-	9300 4600 9300 4250
-Wire Wire Line
-	9400 4050 9400 4600
-Wire Wire Line
-	9500 4150 9500 4600
-Text Label 2450 2600 0    60   ~ 0
+Text Label 2450 3900 0    60   ~ 0
 DWL0
-Text Label 2450 2700 0    60   ~ 0
+Text Label 2450 4000 0    60   ~ 0
 DWL1
-Text Label 2450 2800 0    60   ~ 0
+Text Label 2450 4100 0    60   ~ 0
 DWL2
-Text Label 2450 2900 0    60   ~ 0
+Text Label 2450 4200 0    60   ~ 0
 DWL3
 Text Label 4850 1900 2    60   ~ 0
@@
 Text Label 8250 1850 0    60   ~ 0
 AD_CLK
-Text Label 8300 4150 1    60   ~ 0
+Text Label 2450 2150 0    60   ~ 0
 DWL0
-Text Label 8200 4150 1    60   ~ 0
+Text Label 2450 2250 0    60   ~ 0
 DWL1
-Text Label 8100 4150 1    60   ~ 0
+Text Label 2450 2350 0    60   ~ 0
 DWL2
-Text Label 8000 4150 1    60   ~ 0
+Text Label 2450 2450 0    60   ~ 0
 DWL3
-Text Label 9300 4250 1    60   ~ 0
-SSR_ON
-Text Label 8500 4250 1    60   ~ 0
+Text Label 2450 1850 0    60   ~ 0
 T_SCK
-Text Label 8400 4250 1    60   ~ 0
+Text Label 2450 1950 0    60   ~ 0
 T_SIO
-Text Label 8600 4250 1    60   ~ 0
+Text Label 2450 1750 0    60   ~ 0
 T_CS
-Text Label 8700 4250 1    60   ~ 0
+Text Label 2450 1550 0    60   ~ 0
 AD_CS
-Text Label 8900 4250 1    60   ~ 0
+Text Label 2450 1450 0    60   ~ 0
 AD_MOSI
-Text Label 9000 4250 1    60   ~ 0
+Text Label 2450 1350 0    60   ~ 0
 AD_MISO
-Text Label 9200 4250 1    60   ~ 0
+Text Label 2450 1250 0    60   ~ 0
 AD_CLK
 Wire Wire Line
@@
 Wire Wire Line
 	7050 1150 6100 1150
-Wire Wire Line
-	8700 4600 8700 4250
-Wire Wire Line
-	8400 4600 8400 4250
 $Comp
 L CONN_01X03 POWER1
@@
 Text GLabel 3050 6050 1    60   Input ~ 0
 230V_NEUTRAL
-Text Label 6100 1900 0    60   ~ 0
-MOTOR+
 Text Label 3350 5900 0    60   ~ 0
 MOTOR+
@@
 Text GLabel 2950 6050 1    60   Input ~ 0
 230V_GND
-Text Notes 7500 6150 0    60   ~ 0
-Embedded Control Computer
-Text GLabel 9700 5100 3    60   Input ~ 0
-GND
-Text GLabel 7800 5100 3    60   Input ~ 0
-GND
-Text GLabel 7900 4600 1    60   Input ~ 0
-+5V
 $Comp
 L R R2
@@
 Wire Wire Line
 	9850 3600 9850 3750
-Wire Wire Line
-	9600 4600 9600 4250
 $Comp
 L R R1
@@
 Text Label 6800 4300 3    60   ~ 0
 DWL0
-Text Label 8300 5400 3    60   ~ 0
-DWL3
-Text Label 8400 5400 3    60   ~ 0
-DWL2
-Text Label 8500 5400 3    60   ~ 0
-DWL1
-Text Label 8600 5400 3    60   ~ 0
-DWL0
-Text GLabel 7900 5700 3    60   Input ~ 0
-+3.3V
 $Sheet
-S 1300 1000 1550 1150
+S 1300 1000 1150 1950
 U 599A5341
 F0 "system_on_module" 60
 F1 "system_on_module.sch" 60
+F2 "SSR_ON" I R 2450 1100 60
+F3 "AD_CLK" I R 2450 1250 60
+F4 "AD_MISO" I R 2450 1350 60
+F5 "AD_MOSI" I R 2450 1450 60
+F6 "AD_CS" I R 2450 1550 60
+F7 "TEMPERATURE_CS" I R 2450 1750 60
+F8 "TEMPERATURE_SCK" I R 2450 1850 60
+F9 "TEMPERATURE_SIO" I R 2450 1950 60
+F10 "WATER_LEVEL0" I R 2450 2150 60
+F11 "WATER_LEVEL1" I R 2450 2250 60
+F12 "WATER_LEVEL2" I R 2450 2350 60
+F13 "WATER_LEVEL3" I R 2450 2450 60
+F14 "INDICATOR_LED_0" I R 2450 2600 60
+F15 "INDICATOR_LED_1" I R 2450 2700 60
+F16 "INDICATOR_LED_2" I R 2450 2800 60
 $EndSheet
+Text Label 6100 1900 0    60   ~ 0
+MOTOR+
+Text Label 2450 1100 0    60   ~ 0
+SSR_ON
+Text Label 2450 2600 0    60   ~ 0
+INDICATOR_LED_0
+Text Label 2450 2700 0    60   ~ 0
+INDICATOR_LED_1
+Text Label 2450 2800 0    60   ~ 0
+INDICATOR_LED_2
+Text Label 9400 4050 2    60   ~ 0
+INDICATOR_LED_0
+Text Label 9500 4150 2    60   ~ 0
+INDICATOR_LED_1
+Text Label 9600 4250 2    60   ~ 0
+INDICATOR_LED_2
 $EndSCHEMATC
